File: ReminderTracker.kicad_sch (KiCad schematic)
At the start: 21 parts, among them J1 External RTC, SW1 SW_Push, SW2 SW_Push, SW3 SW_Push, SW4 SW_Push, SW5 SW_Push, SW6 SW_Push, U1 XIAO-ESP32-C3-DIP

Commit message: R1
Parts:
- C1: now not fitted; now left out of the parts list
Connections:
- net +3.3V: now also C5.1, C6.1, C7.1, D4.1 (VDD), D5.1 (VDD), D6.1 (VDD)
- net BUTTON_1: now also U1.2 (GPIO3_A1_D1); no longer U1.1 (GPIO2_A0_D0)
- net BUTTON_2: now also U1.3 (GPIO4_A2_D2); no longer U1.2 (GPIO3_A1_D1)
- net BUTTON_3: now also U1.4 (GPIO5_A3_D3); no longer U1.3 (GPIO4_A2_D2)
- net BUTTON_4: now also U1.5 (GPIO6_D4_SDA); no longer U1.4 (GPIO5_A3_D3)
- net BUTTON_5: now also U1.6 (GPIO7_D5_SCL); no longer U1.9 (GPIO8_D8_SCK)
- net BUTTON_6: now also U1.7 (GPIO21_D6_TX); no longer U1.8 (GPIO20_D7_RX)
- net I2C_SCL: now also U1.10 (GPIO9_D9_MISO); no longer U1.6 (GPIO7_D5_SCL)
- net I2C_SDA: now also U1.11 (GPIO10_D10_MOSI); no longer U1.5 (GPIO6_D4_SDA)
- net LED_DATA: now also U1.1 (GPIO2_A0_D0); no longer U1.7 (GPIO21_D6_TX)
Changed lines of the file:
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@@
 	)
 	(junction
+		(at 156.21 21.59)
+		(diameter 0)
+		(color 0 0 0 0)
+	)
+	(junction
 		(at 137.16 21.59)
 		(diameter 0)
@@
 	(wire
 		(pts
-			(xy 146.05 21.59) (xy 156.0349 21.59)
+			(xy 146.05 21.59) (xy 156.21 21.59)
 		)
 		(stroke
@@
 	(global_label "BUTTON_1"
 		(shape input)
-		(at 102.87 74.93 180)
+		(at 102.87 78.74 180)
 		(fields_autoplaced yes)
 		(effects
@@
 		)
 		(property "Intersheetrefs" "${INTERSHEET_REFS}"
-			(at 90.511 74.93 0)
+			(at 90.511 78.74 0)
 			(effects
 				(font
@@
 		)
 	)
+	(global_label "BUTTON_6"
+		(shape input)
+		(at 102.87 97.79 180)
+		(fields_autoplaced yes)
+		(effects
+			(font
+				(size 1.27 1.27)
+			)
+			(justify right)
+		)
+		(property "Intersheetrefs" "${INTERSHEET_REFS}"
+			(at 91.0553 97.79 0)
+			(effects
+				(font
+					(size 1.27 1.27)
+				)
+				(justify right)
+				(hide yes)
+			)
+		)
+	)
 	(global_label "BUTTON_3"
 		(shape input)
@@
 	(global_label "BUTTON_5"
 		(shape input)
-		(at 45.72 93.98 180)
+		(at 102.87 93.98 180)
 		(fields_autoplaced yes)
 		(effects
@@
 		)
 		(property "Intersheetrefs" "${INTERSHEET_REFS}"
-			(at 34.3286 93.98 0)
+			(at 90.511 93.98 0)
 			(effects
 				(font
@@
 		)
 	)
-	(global_label "BUTTON_4"
+	(global_label "BUTTON_5"
 		(shape input)
-		(at 102.87 86.36 180)
+		(at 45.72 93.98 180)
 		(fields_autoplaced yes)
 		(effects
@@
 		)
 		(property "Intersheetrefs" "${INTERSHEET_REFS}"
-			(at 90.511 86.36 0)
+			(at 34.3286 93.98 0)
 			(effects
 				(font
@@
 		)
 	)
-	(global_label "I2C_SCL"
-		(shape bidirectional)
-		(at 200.66 72.39 0)
+	(global_label "BUTTON_4"
+		(shape input)
+		(at 102.87 90.17 180)
 		(fields_autoplaced yes)
 		(effects
@@
 				(size 1.27 1.27)
 			)
-			(justify left)
+			(justify right)
 		)
 		(property "Intersheetrefs" "${INTERSHEET_REFS}"
-			(at 212.316 72.39 0)
+			(at 91.4786 90.17 0)
 			(effects
 				(font
 					(size 1.27 1.27)
 				)
-				(justify left)
+				(justify right)
 				(hide yes)
 			)
 		)
 	)
-	(global_label "BUTTON_5"
-		(shape input)
-		(at 140.97 93.98 0)
+	(global_label "I2C_SDA"
+		(shape bidirectional)
+		(at 140.97 86.36 0)
 		(fields_autoplaced yes)
 		(effects
@@
 		)
 		(property "Intersheetrefs" "${INTERSHEET_REFS}"
-			(at 152.3614 93.98 0)
+			(at 152.6865 86.36 0)
 			(effects
 				(font
@@
 		)
 	)
-	(global_label "I2C_SDA"
+	(global_label "I2C_SCL"
 		(shape bidirectional)
-		(at 102.87 90.17 180)
+		(at 200.66 72.39 0)
 		(fields_autoplaced yes)
 		(effects
@@
 				(size 1.27 1.27)
 			)
-			(justify right)
+			(justify left)
 		)
 		(property "Intersheetrefs" "${INTERSHEET_REFS}"
-			(at 91.1535 90.17 0)
+			(at 212.316 72.39 0)
 			(effects
 				(font
 					(size 1.27 1.27)
 				)
-				(justify right)
+				(justify left)
 				(hide yes)
 			)
@@
 	(global_label "BUTTON_3"
 		(shape input)
-		(at 102.87 82.55 180)
+		(at 102.87 86.36 180)
 		(fields_autoplaced yes)
 		(effects
@@
 		)
 		(property "Intersheetrefs" "${INTERSHEET_REFS}"
-			(at 90.511 82.55 0)
+			(at 90.511 86.36 0)
 			(effects
 				(font
@@
 		)
 	)
-	(global_label "I2C_SCL"
-		(shape bidirectional)
-		(at 102.87 93.98 180)
-		(fields_autoplaced yes)
-		(effects
-			(font
-				(size 1.27 1.27)
-			)
-			(justify right)
-		)
-		(property "Intersheetrefs" "${INTERSHEET_REFS}"
-			(at 91.214 93.98 0)
-			(effects
-				(font
-					(size 1.27 1.27)
-				)
-				(justify right)
-				(hide yes)
-			)
-		)
-	)
 	(global_label "BUTTON_2"
 		(shape input)
-		(at 102.87 78.74 180)
+		(at 102.87 82.55 180)
 		(fields_autoplaced yes)
 		(effects
@@
 		)
 		(property "Intersheetrefs" "${INTERSHEET_REFS}"
-			(at 90.511 78.74 0)
+			(at 90.511 82.55 0)
 			(effects
 				(font
@@
 		)
 	)
-	(global_label "BUTTON_6"
-		(shape input)
-		(at 140.97 97.79 0)
+	(global_label "I2C_SCL"
+		(shape bidirectional)
+		(at 140.97 90.17 0)
 		(fields_autoplaced yes)
 		(effects
@@
 		)
 		(property "Intersheetrefs" "${INTERSHEET_REFS}"
-			(at 153.329 97.79 0)
+			(at 152.626 90.17 0)
 			(effects
 				(font
@@
 	(global_label "LED_DATA"
 		(shape output)
-		(at 102.87 97.79 180)
+		(at 102.87 74.93 180)
 		(fields_autoplaced yes)
 		(effects
@@
 		)
 		(property "Intersheetrefs" "${INTERSHEET_REFS}"
-			(at 91.0553 97.79 0)
+			(at 90.511 74.93 0)
 			(effects
 				(font
@@
 		(unit 1)
 		(exclude_from_sim no)
-		(in_bom yes)
-		(on_board yes)
-		(dnp no)
+		(in_bom no)
+		(on_board no)
+		(dnp yes)
 		(property "Reference" "C1"
 			(at 85.09 22.8662 0)
